Commit message: [Add] モデルをrviz上で出すところまで

File: nachi_description/robots/mz07/mz07.urdf.xacro (robot description, xacro)
@@ -1,4 +1,4 @@
 <?xml version="1.0"?>
-<robot name="sia5" xmlns:xacro="http://ros.org/wiki/xacro">
+<robot name="mz07" xmlns:xacro="http://ros.org/wiki/xacro">
   <xacro:include filename="$(find nachi_description)/urdf/common.xacro" />
   <xacro:include filename="$(find nachi_description)/urdf/materials.xacro" />
@@ -6,5 +6,20 @@
   <xacro:property name="J1_upper_limit" value="${170*M_PI/180.0}"/>
   <xacro:property name="J1_lower_limit" value="-${J1_upper_limit}"/>
- <xacro:property name="J1_velocity_limit" value="${450.0*M_PI/180.0}"/>
+  <xacro:property name="J2_upper_limit" value="${80*M_PI/180.0}"/>
+  <xacro:property name="J2_lower_limit" value="${-135*M_PI/180.0}"/>
+  <xacro:property name="J3_upper_limit" value="${90*M_PI/180.0}"/>
+  <xacro:property name="J3_lower_limit" value="${-135*M_PI/180.0}"/>
+  <xacro:property name="J4_upper_limit" value="${190*M_PI/180.0}"/>
+  <xacro:property name="J4_lower_limit" value="-${J4_upper_limit}"/>
+  <xacro:property name="J5_upper_limit" value="${120*M_PI/180.0}"/>
+  <xacro:property name="J5_lower_limit" value="-${J5_upper_limit}"/>
+  <xacro:property name="J6_upper_limit" value="${360*M_PI/180.0}"/>
+  <xacro:property name="J6_lower_limit" value="-${J6_upper_limit}"/>
+  <xacro:property name="J1_velocity_limit" value="${450.0*M_PI/180.0}"/>
+  <xacro:property name="J2_velocity_limit" value="${380.0*M_PI/180.0}"/>
+  <xacro:property name="J3_velocity_limit" value="${520.0*M_PI/180.0}"/>
+  <xacro:property name="J4_velocity_limit" value="${550.0*M_PI/180.0}"/>
+  <xacro:property name="J5_velocity_limit" value="${550.0*M_PI/180.0}"/>
+  <xacro:property name="J6_velocity_limit" value="${1000.0*M_PI/180.0}"/>
   <xacro:link_v1 name="base_link" mass="3.0"
            ixx="0.001" ixy="0" ixz="0"
@@ -12,4 +27,24 @@
            izz="0.001"/>
   <xacro:link_v1 name="link_1" mass="3.0"
+           ixx="0.001" ixy="0" ixz="0"
+           iyy="0.001" iyz="0"
+           izz="0.001"/>
+  <xacro:link_v1 name="link_2" mass="3.0"
+           ixx="0.001" ixy="0" ixz="0"
+           iyy="0.001" iyz="0"
+           izz="0.001"/>
+  <xacro:link_v1 name="link_3" mass="3.0"
+           ixx="0.001" ixy="0" ixz="0"
+           iyy="0.001" iyz="0"
+           izz="0.001"/>
+  <xacro:link_v1 name="link_4" mass="3.0"
+           ixx="0.001" ixy="0" ixz="0"
+           iyy="0.001" iyz="0"
+           izz="0.001"/>
+  <xacro:link_v1 name="link_5" mass="3.0"
+           ixx="0.001" ixy="0" ixz="0"
+           iyy="0.001" iyz="0"
+           izz="0.001"/>
+  <xacro:link_v1 name="link_6" mass="3.0"
            ixx="0.001" ixy="0" ixz="0"
            iyy="0.001" iyz="0"
@@ -25,3 +60,53 @@
             skp="1" skv="1"
             sll="${J1_lower_limit}" sul="${J1_upper_limit}"/>
+<xacro:joint_v1 joint_name="J2"
+            parent_name="link_1" child_name="link_2"
+            ox="0.05" oy="0" oz="0.148"
+            roll="0" pitch="0" yaw="0"
+            ax="0" ay="1" az="0"
+            el="30.0"
+            ll="${J2_lower_limit}" ul="${J2_upper_limit}"
+            vl="${J2_velocity_limit}"
+            skp="1" skv="1"
+            sll="${J2_lower_limit}" sul="${J2_upper_limit}"/>
+<xacro:joint_v1 joint_name="J3"
+            parent_name="link_2" child_name="link_3"
+            ox="0" oy="0" oz="0.33"
+            roll="0" pitch="0" yaw="0"
+            ax="0" ay="1" az="0"
+            el="30.0"
+            ll="${J3_lower_limit}" ul="${J3_upper_limit}"
+            vl="${J3_velocity_limit}"
+            skp="1" skv="1"
+            sll="${J3_lower_limit}" sul="${J3_upper_limit}"/>
+<xacro:joint_v1 joint_name="J4"
+            parent_name="link_3" child_name="link_4"
+            ox="0.09" oy="0" oz="0.045"
+            roll="0" pitch="0" yaw="0"
+            ax="1" ay="0" az="0"
+            el="30.0"
+            ll="${J4_lower_limit}" ul="${J4_upper_limit}"
+            vl="${J4_velocity_limit}"
+            skp="1" skv="1"
+            sll="${J4_lower_limit}" sul="${J4_upper_limit}"/>
+<xacro:joint_v1 joint_name="J5"
+            parent_name="link_4" child_name="link_5"
+            ox="0.25" oy="0" oz="0"
+            roll="0" pitch="0" yaw="0"
+            ax="0" ay="1" az="0"
+            el="30.0"
+            ll="${J5_lower_limit}" ul="${J5_upper_limit}"
+            vl="${J5_velocity_limit}"
+            skp="1" skv="1"
+            sll="${J5_lower_limit}" sul="${J5_upper_limit}"/>
+<xacro:joint_v1 joint_name="J6"
+            parent_name="link_5" child_name="link_6"
+            ox="0.063" oy="0" oz="0"
+            roll="0" pitch="0" yaw="0"
+            ax="1" ay="0" az="0"
+            el="30.0"
+            ll="${J6_lower_limit}" ul="${J6_upper_limit}"
+            vl="${J6_velocity_limit}"
+            skp="1" skv="1"
+            sll="${J6_lower_limit}" sul="${J6_upper_limit}"/>
 </robot>

Commit message: [Fix] 限界角度のリミット修正

File: nachi_description/robots/mz07/mz07.urdf.xacro (robot description, xacro)
@@ -6,8 +6,8 @@
   <xacro:property name="J1_upper_limit" value="${170*M_PI/180.0}"/>
   <xacro:property name="J1_lower_limit" value="-${J1_upper_limit}"/>
-  <xacro:property name="J2_upper_limit" value="${80*M_PI/180.0}"/>
-  <xacro:property name="J2_lower_limit" value="${-135*M_PI/180.0}"/>
-  <xacro:property name="J3_upper_limit" value="${90*M_PI/180.0}"/>
-  <xacro:property name="J3_lower_limit" value="${-135*M_PI/180.0}"/>
+  <xacro:property name="J2_upper_limit" value="${135*M_PI/180.0}"/>
+  <xacro:property name="J2_lower_limit" value="${-80*M_PI/180.0}"/>
+  <xacro:property name="J3_upper_limit" value="${46*M_PI/180.0}"/>
+  <xacro:property name="J3_lower_limit" value="${-180*M_PI/180.0}"/>
   <xacro:property name="J4_upper_limit" value="${190*M_PI/180.0}"/>
   <xacro:property name="J4_lower_limit" value="-${J4_upper_limit}"/>
@@ -22,4 +22,5 @@
   <xacro:property name="J5_velocity_limit" value="${550.0*M_PI/180.0}"/>
   <xacro:property name="J6_velocity_limit" value="${1000.0*M_PI/180.0}"/>
+  <link name="world"/>
   <xacro:link_v1 name="base_link" mass="3.0"
            ixx="0.001" ixy="0" ixz="0"
@@ -50,63 +51,73 @@
            iyy="0.001" iyz="0"
            izz="0.001"/>
-<xacro:joint_v1 joint_name="J1"
-            parent_name="base_link" child_name="link_1"
-            ox="0" oy="0" oz="0.197"
-            roll="0" pitch="0" yaw="0"
-            ax="0" ay="0" az="1"
-            el="30.0"
-            ll="${J1_lower_limit}" ul="${J1_upper_limit}"
-            vl="${J1_velocity_limit}"
-            skp="1" skv="1"
-            sll="${J1_lower_limit}" sul="${J1_upper_limit}"/>
-<xacro:joint_v1 joint_name="J2"
-            parent_name="link_1" child_name="link_2"
-            ox="0.05" oy="0" oz="0.148"
-            roll="0" pitch="0" yaw="0"
-            ax="0" ay="1" az="0"
-            el="30.0"
-            ll="${J2_lower_limit}" ul="${J2_upper_limit}"
-            vl="${J2_velocity_limit}"
-            skp="1" skv="1"
-            sll="${J2_lower_limit}" sul="${J2_upper_limit}"/>
-<xacro:joint_v1 joint_name="J3"
-            parent_name="link_2" child_name="link_3"
-            ox="0" oy="0" oz="0.33"
-            roll="0" pitch="0" yaw="0"
-            ax="0" ay="1" az="0"
-            el="30.0"
-            ll="${J3_lower_limit}" ul="${J3_upper_limit}"
-            vl="${J3_velocity_limit}"
-            skp="1" skv="1"
-            sll="${J3_lower_limit}" sul="${J3_upper_limit}"/>
-<xacro:joint_v1 joint_name="J4"
-            parent_name="link_3" child_name="link_4"
-            ox="0.09" oy="0" oz="0.045"
-            roll="0" pitch="0" yaw="0"
-            ax="1" ay="0" az="0"
-            el="30.0"
-            ll="${J4_lower_limit}" ul="${J4_upper_limit}"
-            vl="${J4_velocity_limit}"
-            skp="1" skv="1"
-            sll="${J4_lower_limit}" sul="${J4_upper_limit}"/>
-<xacro:joint_v1 joint_name="J5"
-            parent_name="link_4" child_name="link_5"
-            ox="0.25" oy="0" oz="0"
-            roll="0" pitch="0" yaw="0"
-            ax="0" ay="1" az="0"
-            el="30.0"
-            ll="${J5_lower_limit}" ul="${J5_upper_limit}"
-            vl="${J5_velocity_limit}"
-            skp="1" skv="1"
-            sll="${J5_lower_limit}" sul="${J5_upper_limit}"/>
-<xacro:joint_v1 joint_name="J6"
-            parent_name="link_5" child_name="link_6"
-            ox="0.063" oy="0" oz="0"
-            roll="0" pitch="0" yaw="0"
-            ax="1" ay="0" az="0"
-            el="30.0"
-            ll="${J6_lower_limit}" ul="${J6_upper_limit}"
-            vl="${J6_velocity_limit}"
-            skp="1" skv="1"
-            sll="${J6_lower_limit}" sul="${J6_upper_limit}"/>
+  <link name="tool0"/>
+  <joint name="world" type="fixed">
+    <parent link="world"/>
+    <child link="base_link"/>
+  </joint>
+  <xacro:joint_v1 joint_name="J1"
+                 parent_name="base_link" child_name="link_1"
+                 ox="0" oy="0" oz="0.197"
+                 roll="0" pitch="0" yaw="0"
+                 ax="0" ay="0" az="1"
+                 el="30.0"
+                 ll="${J1_lower_limit}" ul="${J1_upper_limit}"
+                 vl="${J1_velocity_limit}"
+                 skp="1" skv="1"
+                 sll="${J1_lower_limit}" sul="${J1_upper_limit}"/>
+  <xacro:joint_v1 joint_name="J2"
+                 parent_name="link_1" child_name="link_2"
+                 ox="0.05" oy="0" oz="0.148"
+                 roll="0" pitch="0" yaw="0"
+                 ax="0" ay="1" az="0"
+                 el="30.0"
+                 ll="${J2_lower_limit}" ul="${J2_upper_limit}"
+                 vl="${J2_velocity_limit}"
+                 skp="1" skv="1"
+                 sll="${J2_lower_limit}" sul="${J2_upper_limit}"/>
+  <xacro:joint_v1 joint_name="J3"
+                 parent_name="link_2" child_name="link_3"
+                 ox="0" oy="0" oz="0.33"
+                 roll="0" pitch="0" yaw="0"
+                 ax="0" ay="1" az="0"
+                 el="30.0"
+                 ll="${J3_lower_limit}" ul="${J3_upper_limit}"
+                 vl="${J3_velocity_limit}"
+                 skp="1" skv="1"
+                 sll="${J3_lower_limit}" sul="${J3_upper_limit}"/>
+  <xacro:joint_v1 joint_name="J4"
+                 parent_name="link_3" child_name="link_4"
+                 ox="0.09" oy="0" oz="0.045"
+                 roll="0" pitch="0" yaw="0"
+                 ax="1" ay="0" az="0"
+                 el="30.0"
+                 ll="${J4_lower_limit}" ul="${J4_upper_limit}"
+                 vl="${J4_velocity_limit}"
+                 skp="1" skv="1"
+                 sll="${J4_lower_limit}" sul="${J4_upper_limit}"/>
+  <xacro:joint_v1 joint_name="J5"
+                 parent_name="link_4" child_name="link_5"
+                 ox="0.25" oy="0" oz="0"
+                 roll="0" pitch="0" yaw="0"
+                 ax="0" ay="1" az="0"
+                 el="30.0"
+                 ll="${J5_lower_limit}" ul="${J5_upper_limit}"
+                 vl="${J5_velocity_limit}"
+                 skp="1" skv="1"
+                 sll="${J5_lower_limit}" sul="${J5_upper_limit}"/>
+  <xacro:joint_v1 joint_name="J6"
+                 parent_name="link_5" child_name="link_6"
+                 ox="0.063" oy="0" oz="0"
+                 roll="0" pitch="0" yaw="0"
+                 ax="1" ay="0" az="0"
+                 el="30.0"
+                 ll="${J6_lower_limit}" ul="${J6_upper_limit}"
+                 vl="${J6_velocity_limit}"
+                 skp="1" skv="1"
+                 sll="${J6_lower_limit}" sul="${J6_upper_limit}"/>
+  <joint name="joint_tool0" type="fixed">
+    <origin rpy="0 0 0" xyz="0.0195 0 0"/>
+    <parent link="link_6"/>
+    <child link="tool0"/>
+  </joint>
 </robot>

Commit message: [Update] Solidworksから計算した質量，慣性モーメント情報を追加

File: nachi_description/robots/mz07/mz07.urdf.xacro (robot description, xacro)
@@ -29,32 +29,37 @@
   <!-- Link -->
   <link name="world"/>
-  <xacro:link_v1 name="base_link" mass="3.0"
-				 ixx="0.001" ixy="0" ixz="0"
-				 iyy="0.001" iyz="0"
-				 izz="0.001"/>
-  <xacro:link_v1 name="link_1" mass="3.0"
-				 ixx="0.001" ixy="0" ixz="0"
-				 iyy="0.001" iyz="0"
-				 izz="0.001"/>
-  <xacro:link_v1 name="link_2" mass="3.0"
-				 ixx="0.001" ixy="0" ixz="0"
-				 iyy="0.001" iyz="0"
-				 izz="0.001"/>
-  <xacro:link_v1 name="link_3" mass="3.0"
-				 ixx="0.001" ixy="0" ixz="0"
-				 iyy="0.001" iyz="0"
-				 izz="0.001"/>
-  <xacro:link_v1 name="link_4" mass="3.0"
-				 ixx="0.001" ixy="0" ixz="0"
-				 iyy="0.001" iyz="0"
-				 izz="0.001"/>
-  <xacro:link_v1 name="link_5" mass="3.0"
-				 ixx="0.001" ixy="0" ixz="0"
-				 iyy="0.001" iyz="0"
-				 izz="0.001"/>
-  <xacro:link_v1 name="link_6" mass="3.0"
-				 ixx="0.001" ixy="0" ixz="0"
-				 iyy="0.001" iyz="0"
-				 izz="0.001"/>
+  <xacro:link_v1 name="base_link" mass="9.522365"
+				 ixx="0.144495" ixy="-0.000009" ixz="-0.030760"
+				 iyy="0.183352" iyz="-0.000037"
+				 izz="0.079873"/>
+  <xacro:link_v1 name="link_1" mass="5.616960"
+				 ixx="0.087433" ixy="0.000000" ixz="0.013287"
+				 iyy="0.073064" iyz="0.000019"
+				 izz="0.039829"/>
+  <xacro:link_v1 name="link_2" mass="7.350069"
+				 ixx="0.299465" ixy="-0.000010" ixz="-0.012735"
+				 iyy="0.279554" iyz="0.000053"
+				 izz="0.035911"/>
+  <xacro:link_v1 name="link_3" mass="3.724767"
+				 ixx="0.011733" ixy="0.000043" ixz="0.000461"
+				 iyy="0.019531" iyz="0.000024"
+				 izz="0.014154"/>
+  <xacro:link_v1 name="link_4" mass="3.245188"
+				 ixx="0.007141" ixy="0.000562" ixz="0.000255"
+				 iyy="0.054197" iyz="0.000024"
+				 izz="0.056111"/>
+  <xacro:link_v1 name="link_5" mass="0.501938"
+         ixx="0.000539" ixy="0.000001" ixz="0.000000"
+         iyy="0.000892" iyz="-0.000001"
+         izz="0.000962"/>
+  <xacro:link_v1 name="link_6" mass="0.038575"
+         ixx="0.0005" ixy="0.000000" ixz="0.000000"
+         iyy="0.0005" iyz="0.000000"
+         izz="0.0005"/>
+<!--
+  <xacro:link_v1 name="link_6" mass="0.038575"
+				 ixx="0.000027" ixy="0.000000" ixz="0.000000"
+				 iyy="0.000016" iyz="0.000000"
+				 izz="0.000017"/> -->
   <link name="tool0"/>
   <!-- Joint -->

File: nachi_description/robots/mz07/urdf/mz07.urdf (robot description, URDF)
Before this commit: robot mz07, 9 links, 8 joints
Links:
- link base_link: mass 3.0 -> 9.522365
- link link_1: mass 3.0 -> 5.61696
- link link_2: mass 3.0 -> 7.350069
- link link_3: mass 3.0 -> 3.724767
- link link_4: mass 3.0 -> 3.245188
- link link_5: mass 3.0 -> 0.501938
- link link_6: mass 3.0 -> 0.038575
