Commit message: [Fix] Kinectの設置の高さを変更しました

File: nachi_description/robots/mz07/mz07.sensor.urdf.xacro (robot description, xacro)
@@ -11,5 +11,5 @@
   <!-- Joint -->
   <joint name="joint_kinect2" type="fixed">
-    <origin rpy="0 ${10*M_PI/180} ${M_PI}" xyz="1.05024 0 0.8195"/>
+    <origin rpy="0 ${10*M_PI/180} ${M_PI}" xyz="1.5 0 0.4"/>
     <parent link="world"/>
     <child link="kinect2_link"/>

File: nachi_description/robots/mz07/urdf/mz07.sensor.urdf (robot description, URDF)
Before this commit: robot mz07, 11 links, 10 joints
Joints:
- joint joint_kinect2: origin xyz=1.05024 0 0.8195 rpy=0 0.17453293 3.14159274 -> xyz=1.5 0 0.4 rpy=0 0.17453293 3.14159274
