Commit message: Update for migration from indigo to melodic

File: nachi_description/urdf/common.xacro (robot description, xacro)
@@ -1,4 +1,4 @@
 <?xml version="1.0"?>
-<robot>
-  <property name="M_PI" value="3.14159274"/>
+<robot xmlns:xacro="http://ros.org/wiki/xacro">
+  <xacro:property name="M_PI" value="3.14159274"/>
 </robot>
